Commit message: reverted back to non-gazebo rviz setup

File: install/sdp_bot/share/sdp_bot/urdf/all_bot.urdf (robot description, URDF)
Before this commit: robot all_bot, 7 links, 6 joints
Links:
- added link imu_link; collision box size=0.025 0.02 0.0025; visual box size=0.025 0.02 0.0025
Joints:
- added joint imu_joint: type fixed, parent base_link, child imu_link, origin xyz=0 0 0 rpy=0 0 0

File: src/sdp_bot/urdf/all_bot.urdf (robot description, URDF)
Before this commit: robot all_bot, 7 links, 6 joints
Links:
- added link imu_link; collision box size=0.025 0.02 0.0025; visual box size=0.025 0.02 0.0025
Joints:
- added joint imu_joint: type fixed, parent base_link, child imu_link, origin xyz=0 0 0 rpy=0 0 0

Commit message: Erased the front two wheels temporarily

File: install/sdp_bot/share/sdp_bot/urdf/all_bot.urdf (robot description, URDF)
Before this commit: robot all_bot, 8 links, 7 joints
Links:
- removed link front_left_wheel
- removed link front_right_wheel
Joints:
- removed joint base_back_left_wheel_joint
- removed joint base_back_right_wheel_joint
- removed joint base_front_left_wheel_joint
- removed joint base_front_right_wheel_joint
- added joint left_joint: type continuous, parent base_link, child back_left_wheel, origin xyz=-0.060335 0.0635 -0.04572 rpy=0 0 0, axis 0 1 0
- added joint right_joint: type continuous, parent base_link, child back_right_wheel, origin xyz=-0.060335 -0.0635 -0.04572 rpy=0 0 0, axis 0 1 0

Commit message: Revert back to custom control

File: install/sdp_bot/share/sdp_bot/urdf/all_bot.urdf (robot description, URDF)
Before this commit: robot all_bot, 6 links, 5 joints
Links:
- added link front_left_wheel; collision cylinder length=0.0254 radius=0.03175; visual cylinder length=0.0254 radius=0.03175
- added link front_right_wheel; collision cylinder length=0.0254 radius=0.03175; visual cylinder length=0.0254 radius=0.03175
Joints:
- removed joint left_joint
- removed joint right_joint
- added joint base_back_left_wheel_joint: type continuous, parent base_link, child back_left_wheel, origin xyz=-0.060335 0.0635 -0.04572 rpy=0 0 0, axis 0 1 0
- added joint base_back_right_wheel_joint: type continuous, parent base_link, child back_right_wheel, origin xyz=-0.060335 -0.0635 -0.04572 rpy=0 0 0, axis 0 1 0
- added joint base_front_left_wheel_joint: type continuous, parent base_link, child front_left_wheel, origin xyz=0.060335 0.0635 -0.04572 rpy=0 0 0, axis 0 1 0
- added joint base_front_right_wheel_joint: type continuous, parent base_link, child front_right_wheel, origin xyz=0.060335 -0.0635 -0.04572 rpy=0 0 0, axis 0 1 0
